File: W5500_Shield_Ethernet.kicad_pcb (KiCad board)
At the start: 2 copper layers, 47 x 31 mm, 33 parts, among them J1 HR911105A, J2 Conn_02x05_Odd_Even, U2 W5500, Y1 X322525MOB4SI

Commit message: Listo para enviar a jlcpcb
Parts:
- R10: value 49R -> 49.9
- R3, R4, R9: value 50R -> 49.9
- R5, R6, R7, R8: value 3.3R -> 0
- turned U2 to -90 degrees
