File: W5500_Shield_Ethernet.kicad_sch (KiCad schematic)
At the start: 33 parts, among them J1 HR911105A, J2 Conn_02x05_Odd_Even, U2 W5500, Y1 X322525MOB4SI

Commit message: Listo para enviar a jlcpcb
Parts:
- R10: value 49R -> 49.9
- R3, R4, R9: value 50R -> 49.9
- R5, R6, R7, R8: value 3.3R -> 0
Changed lines of the file:
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@@
     (in_bom yes) (on_board yes)
     (property "Reference" "R5" (id 0) (at 123.825 52.705 90))
-    (property "Value" "3.3R" (id 1) (at 123.825 55.245 90))
+    (property "Value" "0" (id 1) (at 123.825 55.245 90))
     (property "Footprint" "Resistor_SMD:R_0402_1005Metric" (id 2) (at 123.825 57.023 90)
       (effects (font (size 1.27 1.27)) hide)
@@
     (in_bom yes) (on_board yes)
     (property "Reference" "R9" (id 0) (at 136.525 71.755 90))
-    (property "Value" "50R" (id 1) (at 133.985 71.755 90))
+    (property "Value" "49.9" (id 1) (at 133.985 71.755 90))
     (property "Footprint" "Resistor_SMD:R_0402_1005Metric" (id 2) (at 132.207 71.755 90)
       (effects (font (size 1.27 1.27)) hide)
@@
     (in_bom yes) (on_board yes)
     (property "Reference" "R6" (id 0) (at 120.015 59.69 90))
-    (property "Value" "3.3R" (id 1) (at 123.825 57.785 90))
+    (property "Value" "0" (id 1) (at 123.825 57.785 90))
     (property "Footprint" "Resistor_SMD:R_0402_1005Metric" (id 2) (at 123.825 59.563 90)
       (effects (font (size 1.27 1.27)) hide)
@@
     (in_bom yes) (on_board yes)
     (property "Reference" "R10" (id 0) (at 142.875 71.755 90))
-    (property "Value" "49R" (id 1) (at 140.335 71.755 90))
+    (property "Value" "49.9" (id 1) (at 140.335 71.755 90))
     (property "Footprint" "Resistor_SMD:R_0402_1005Metric" (id 2) (at 138.557 71.755 90)
       (effects (font (size 1.27 1.27)) hide)
@@
     (in_bom yes) (on_board yes)
     (property "Reference" "R4" (id 0) (at 140.97 48.895 90))
-    (property "Value" "50R" (id 1) (at 143.51 48.895 90))
+    (property "Value" "49.9" (id 1) (at 143.51 48.895 90))
     (property "Footprint" "Resistor_SMD:R_0402_1005Metric" (id 2) (at 145.288 48.895 90)
       (effects (font (size 1.27 1.27)) hide)
@@
   (symbol (lib_id "Device:C_Small") (at 55.245 97.79 0) (unit 1)
     (in_bom yes) (on_board yes)
-    (property "Reference" "C12" (id 0) (at 50.8 97.155 0)
+    (property "Reference" "C12" (id 0) (at 48.895 96.52 0)
       (effects (font (size 1.27 1.27)) (justify left))
     )
@@
     (in_bom yes) (on_board yes)
     (property "Reference" "R8" (id 0) (at 120.015 67.31 90))
-    (property "Value" "3.3R" (id 1) (at 123.825 65.405 90))
+    (property "Value" "0" (id 1) (at 123.825 65.405 90))
     (property "Footprint" "Resistor_SMD:R_0402_1005Metric" (id 2) (at 123.825 67.183 90)
       (effects (font (size 1.27 1.27)) hide)
@@
     (in_bom yes) (on_board yes)
     (property "Reference" "R7" (id 0) (at 123.825 60.325 90))
-    (property "Value" "3.3R" (id 1) (at 123.825 62.865 90))
+    (property "Value" "0" (id 1) (at 123.825 62.865 90))
     (property "Footprint" "Resistor_SMD:R_0402_1005Metric" (id 2) (at 123.825 64.643 90)
       (effects (font (size 1.27 1.27)) hide)
@@
     (in_bom yes) (on_board yes)
     (property "Reference" "R3" (id 0) (at 134.62 48.895 90))
-    (property "Value" "50R" (id 1) (at 137.16 48.895 90))
+    (property "Value" "49.9" (id 1) (at 137.16 48.895 90))
     (property "Footprint" "Resistor_SMD:R_0402_1005Metric" (id 2) (at 138.938 48.895 90)
       (effects (font (size 1.27 1.27)) hide)
@@
     )
     (path "/fb546fa0-9905-46be-b6f1-aaecdc75e1c4"
-      (reference "R3") (unit 1) (value "50R") (footprint "Resistor_SMD:R_0402_1005Metric")
+      (reference "R3") (unit 1) (value "49.9") (footprint "Resistor_SMD:R_0402_1005Metric")
     )
     (path "/4b779a94-05df-4176-a8e8-6fd07c8ad08b"
-      (reference "R4") (unit 1) (value "50R") (footprint "Resistor_SMD:R_0402_1005Metric")
+      (reference "R4") (unit 1) (value "49.9") (footprint "Resistor_SMD:R_0402_1005Metric")
     )
     (path "/1afc99a2-a1b8-4fc7-9c93-398e002f4126"
-      (reference "R5") (unit 1) (value "3.3R") (footprint "Resistor_SMD:R_0402_1005Metric")
+      (reference "R5") (unit 1) (value "0") (footprint "Resistor_SMD:R_0402_1005Metric")
     )
     (path "/3819be28-f917-4f88-9fb0-92f88eecc34a"
-      (reference "R6") (unit 1) (value "3.3R") (footprint "Resistor_SMD:R_0402_1005Metric")
+      (reference "R6") (unit 1) (value "0") (footprint "Resistor_SMD:R_0402_1005Metric")
     )
     (path "/f9e5bea8-4844-4f9d-be09-e86dd96baefe"
-      (reference "R7") (unit 1) (value "3.3R") (footprint "Resistor_SMD:R_0402_1005Metric")
+      (reference "R7") (unit 1) (value "0") (footprint "Resistor_SMD:R_0402_1005Metric")
     )
     (path "/8ebe8738-16bb-4671-8e8b-6e62436fa20c"
-      (reference "R8") (unit 1) (value "3.3R") (footprint "Resistor_SMD:R_0402_1005Metric")
+      (reference "R8") (unit 1) (value "0") (footprint "Resistor_SMD:R_0402_1005Metric")
     )
     (path "/343d4240-ae68-4cfe-911f-cd40fbcae535"
-      (reference "R9") (unit 1) (value "50R") (footprint "Resistor_SMD:R_0402_1005Metric")
+      (reference "R9") (unit 1) (value "49.9") (footprint "Resistor_SMD:R_0402_1005Metric")
     )
     (path "/3c12e23f-6423-49d7-b43d-84644a3eac91"
-      (reference "R10") (unit 1) (value "49R") (footprint "Resistor_SMD:R_0402_1005Metric")
+      (reference "R10") (unit 1) (value "49.9") (footprint "Resistor_SMD:R_0402_1005Metric")
     )
     (path "/aca347b8-4846-4ef3-a3ac-4214b95eb178"
